File: PCB/seed75.kicad_pcb (KiCad board)
At the start: 2 copper layers, 317.8 x 133.5 mm, 172 parts, among them J1 Conn_01x06_Pin, SW1 SW_Push, SW10 SW_Push, SW11 SW_Push, SW12 SW_Push, SW13 SW_Push, SW14 SW_Push, SW15 RotaryEncoder_Switch, SW16 SW_Push, SW17 SW_Push, SW18 SW_Push, SW19 SW_Push, SW2 SW_Push, SW20 SW_Push, SW21 SW_Push, SW22 SW_Push, SW23 SW_Push, SW24 SW_Push, SW25 SW_Push, SW26 SW_Push, SW27 SW_Push, SW28 SW_Push, SW29 SW_Push, SW3 SW_Push, SW30 SW_Push, SW31 SW_Push, SW32 SW_Push, SW33 SW_Push, SW34 SW_Push, SW35 SW_Push, SW36 SW_Push, SW37 SW_Push, SW38 SW_Push, SW39 SW_Push, SW4 SW_Push, SW40 SW_Push, SW41 SW_Push, SW42 SW_Push, SW43 SW_Push, SW44 SW_Push, SW45 SW_Push, SW46 SW_Push, SW47 SW_Push, SW48 SW_Push, SW49 SW_Push, SW5 SW_Push, SW50 SW_Push, SW51 SW_Push, SW52 SW_Push, SW53 SW_Push, SW54 SW_Push, SW55 SW_Push, SW56 SW_Push, SW57 SW_Push, SW58 SW_Push, SW59 SW_Push, SW6 SW_Push, SW60 SW_Push, SW61 SW_Push, SW62 SW_Push, SW63 SW_Push, SW64 SW_Push, SW65 SW_Push, SW66 SW_Push, SW67 SW_Push, SW68 SW_Push, SW69 SW_Push, SW7 SW_Push, SW70 SW_Push, SW71 SW_Push, SW72 SW_Push, SW73 SW_Push, SW74 SW_Push, SW75 SW_Push, SW76 SW_Push, SW77 SW_Push, SW78 SW_Push, SW79 SW_Push, SW8 SW_Push, SW80 SW_Push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

Commit message: feat: fixed to pcb
Parts:
- A1: footprint Module:RaspberryPi_Pico_Common_Unspecified -> ScottoKeebs_MCU:Raspberry_Pi_Pico
- SW1, SW10, SW11, SW12, SW13, SW14, SW16, SW17, SW18, SW19, SW2, SW20, SW21, SW22, SW23, SW24, SW25, SW26, SW27, SW28, SW3, SW30, SW32, SW33, SW34, SW35, SW36, SW37, SW38, SW39, SW4, SW40, SW41, SW42, SW43, SW45, SW47, SW48, SW49, SW5, SW50, SW51, SW52, SW53, SW54, SW55, SW56, SW57, SW59, SW6, SW61, SW62, SW63, SW64, SW65, SW66, SW67, SW68, SW69, SW7, SW70, SW72, SW73, SW78, SW79, SW8, SW80, SW81, SW82, SW83, SW9: footprint PCM_Switch_Keyboard_Hotswap_Kailh:SW_Hotswap_Kailh_MX_Plated_1.00u_With_Switch -> CF_Switch_MX_Hotswap:SW_Hotswap_Kailh_MX_Plated_1.00u_With_Switch
- SW29: footprint PCM_Switch_Keyboard_Hotswap_Kailh:SW_Hotswap_Kailh_MX_Plated_2.00u_With_switch -> CF_Switch_MX_Hotswap:SW_Hotswap_Kailh_MX_Plated_2.00u_With_Switch
- SW31, SW44: footprint PCM_Switch_Keyboard_Hotswap_Kailh:SW_Hotswap_Kailh_MX_Plated_1.50u_With_Switch -> CF_Switch_MX_Hotswap:SW_Hotswap_Kailh_MX_Plated_1.50u_With_Switch
- SW46, SW71: footprint PCM_Switch_Keyboard_Hotswap_Kailh:SW_Hotswap_Kailh_MX_Plated_1.75u_With_Switch -> CF_Switch_MX_Hotswap:SW_Hotswap_Kailh_MX_Plated_1.75u_With_Switch
- SW58, SW60: footprint PCM_Switch_Keyboard_Hotswap_Kailh:SW_Hotswap_Kailh_MX_Plated_2.25u_With_Switch -> CF_Switch_MX_Hotswap:SW_Hotswap_Kailh_MX_Plated_2.25u_With_Switch
- SW74, SW75, SW76: footprint PCM_Switch_Keyboard_Hotswap_Kailh:SW_Hotswap_Kailh_MX_Plated_1.25u_With_Switch -> CF_Switch_MX_Hotswap:SW_Hotswap_Kailh_MX_Plated_1.25u_With_Switch
- SW77: footprint PCM_Switch_Keyboard_Hotswap_Kailh:SW_Hotswap_Kailh_MX_Plated_6.25u_With_Switch -> CF_Switch_MX_Hotswap:SW_Hotswap_Kailh_MX_Plated_6.25u_With_Switch
- moved A1 1.00 mm to (90.9, 52.5)
Routing:
- net Row 0: track 311.7 -> 316.5 mm
- net VSYS: track 71.3 -> 76.0 mm, vias 0 -> 2
- net Row 2: track 370.8 -> 374.9 mm, vias 0 -> 1
- net Row 4: track 404.7 -> 408.4 mm, vias 0 -> 4
- net Row 5: track 421.2 -> 418.2 mm, vias 0 -> 2
- net Row 3: track 386.7 -> 389.1 mm
- net Col 2: track 127.2 -> 129.4 mm
- net GPIO27_ABC1: track 86.8 -> 89.0 mm, vias 2 -> 0
- net Col 13: track 382.3 -> 380.5 mm
- net Row 1: track 314.5 -> 316.3 mm
- net Col 1: track 139.5 -> 141.0 mm, vias 0 -> 1
- net RE_B: track 254.2 -> 253.0 mm
- net Col 0: track 117.5 -> 118.6 mm
- net 3v3: track 65.7 -> 66.8 mm, vias 2 -> 3
- net GPIO26_ABC0: track 90.8 -> 91.8 mm, vias 2 -> 0
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
Commit message: fix: pcb changes
Other:
- board text added: "Seed75"
- board text added: "github.com/ikrishagarwal"
